File: PCB/X0chimilc0/Audio_IO.sch (KiCad schematic (older format))
At the start: 0 parts

Commit message: USB C DDR3L MCU
more with MCU and USB C and DDR3L
Parts:
- added T? (x2): ACJS-MHDC, AVR-KiCAD-Lib-Connectors:ACJS-MHDC, symbol AVR-KiCAD-Lib-Connectors:ACJS-MHDC
- added T?: ACJS-MHDR, AVR-KiCAD-Lib-Connectors:ACJS-MHDR, symbol AVR-KiCAD-Lib-Connectors:ACJS-MHDR
Changed lines of the file:
@@
 $Descr A4 11693 8268
 encoding utf-8
-Sheet 1 10
+Sheet 9 11
 Title ""
 Date ""
@@
 Comment4 ""
 $EndDescr
+$Comp
+L AVR-KiCAD-Lib-Connectors:ACJS-MHDC T?
+U 1 1 5E9F6D6F
+P 3850 2150
+F 0 "T?" H 3583 3175 50  0000 C CNN
+F 1 "ACJS-MHDC" H 3583 3084 50  0000 C CNN
+F 2 "AVR-KiCAD-Lib-Connectors:ACJS-MHDC" H 3650 3700 50  0001 C CNN
+F 3 "http://www.amphenol-sine.com/pdf/datasheet/ACJS-MHDC.pdf" H 3750 3800 50  0001 C CNN
+F 4 "2.83000" H 3200 3150 50  0001 C CNN "Cost QTY: 1"
+F 5 "1.71720" H 3300 3250 50  0001 C CNN "Cost QTY: 1000"
+F 6 "1.61120" H 3400 3350 50  0001 C CNN "Cost QTY: 2500"
+F 7 "*" H 3500 3450 50  0001 C CNN "Cost QTY: 5000"
+F 8 "*" H 3600 3550 50  0001 C CNN "Cost QTY: 10000"
+F 9 "Aphenol Sine Systems Corp" H 3700 3650 50  0001 C CNN "MFR"
+F 10 "ACJS-MHDC" H 3800 3750 50  0001 C CNN "MFR#"
+F 11 "Digikey" H 3900 3850 50  0001 C CNN "Vendor"
+F 12 "889-1816-ND" H 4000 3950 50  0001 C CNN "Vendor #"
+F 13 "AVR" H 4100 4050 50  0001 C CNN "Designer"
+F 14 "29.32mm" H 4200 4150 50  0001 C CNN "Height"
+F 15 "1/1/2019" H 5300 5250 50  0001 C CNN "Date Created"
+F 16 "1/1/2019" H 4300 4250 50  0001 C CNN "Date Modified"
+F 17 "Yes" H 4400 4350 50  0001 C CNN "Lead-Free ?"
+F 18 "RoHS 1" H 4500 4450 50  0001 C CNN "RoHS Levels"
+F 19 "Throughole" H 4600 4550 50  0001 C CNN "Mounting"
+F 20 "12" H 4700 4650 50  0001 C CNN "Pin Count #"
+F 21 "Active" H 4800 4750 50  0001 C CNN "Status"
+F 22 "*" H 4900 4850 50  0001 C CNN "Tolerance"
+F 23 "TRS Stereo Dual Connector " H 5000 4950 50  0001 C CNN "Type"
+F 24 "*" H 5100 5050 50  0001 C CNN "Voltage"
+F 25 "*" H 5200 5200 50  0001 C CNN "Package"
+F 26 "CONN JACK DUAL STEREO 1/4\" R/A" H 5600 5600 50  0001 C CNN "Description"
+F 27 "ACJS-MHDC" H 5400 5400 50  0001 C CNN "_Value_"
+F 28 "*" H 5500 5500 50  0001 C CNN "Management_ID"
+	1    3850 2150
+	1    0    0    -1
+$EndComp
+$Comp
+L AVR-KiCAD-Lib-Connectors:ACJS-MHDC T?
+U 1 1 5E9FB8BE
+P 3900 3950
+F 0 "T?" H 3633 4975 50  0000 C CNN
+F 1 "ACJS-MHDC" H 3633 4884 50  0000 C CNN
+F 2 "AVR-KiCAD-Lib-Connectors:ACJS-MHDC" H 3700 5500 50  0001 C CNN
+F 3 "http://www.amphenol-sine.com/pdf/datasheet/ACJS-MHDC.pdf" H 3800 5600 50  0001 C CNN
+F 4 "2.83000" H 3250 4950 50  0001 C CNN "Cost QTY: 1"
+F 5 "1.71720" H 3350 5050 50  0001 C CNN "Cost QTY: 1000"
+F 6 "1.61120" H 3450 5150 50  0001 C CNN "Cost QTY: 2500"
+F 7 "*" H 3550 5250 50  0001 C CNN "Cost QTY: 5000"
+F 8 "*" H 3650 5350 50  0001 C CNN "Cost QTY: 10000"
+F 9 "Aphenol Sine Systems Corp" H 3750 5450 50  0001 C CNN "MFR"
+F 10 "ACJS-MHDC" H 3850 5550 50  0001 C CNN "MFR#"
+F 11 "Digikey" H 3950 5650 50  0001 C CNN "Vendor"
+F 12 "889-1816-ND" H 4050 5750 50  0001 C CNN "Vendor #"
+F 13 "AVR" H 4150 5850 50  0001 C CNN "Designer"
+F 14 "29.32mm" H 4250 5950 50  0001 C CNN "Height"
+F 15 "1/1/2019" H 5350 7050 50  0001 C CNN "Date Created"
+F 16 "1/1/2019" H 4350 6050 50  0001 C CNN "Date Modified"
+F 17 "Yes" H 4450 6150 50  0001 C CNN "Lead-Free ?"
+F 18 "RoHS 1" H 4550 6250 50  0001 C CNN "RoHS Levels"
+F 19 "Throughole" H 4650 6350 50  0001 C CNN "Mounting"
+F 20 "12" H 4750 6450 50  0001 C CNN "Pin Count #"
+F 21 "Active" H 4850 6550 50  0001 C CNN "Status"
+F 22 "*" H 4950 6650 50  0001 C CNN "Tolerance"
+F 23 "TRS Stereo Dual Connector " H 5050 6750 50  0001 C CNN "Type"
+F 24 "*" H 5150 6850 50  0001 C CNN "Voltage"
+F 25 "*" H 5250 7000 50  0001 C CNN "Package"
+F 26 "CONN JACK DUAL STEREO 1/4\" R/A" H 5650 7400 50  0001 C CNN "Description"
+F 27 "ACJS-MHDC" H 5450 7200 50  0001 C CNN "_Value_"
+F 28 "*" H 5550 7300 50  0001 C CNN "Management_ID"
+	1    3900 3950
+	1    0    0    -1
+$EndComp
+$Comp
+L AVR-KiCAD-Lib-Connectors:ACJS-MHDR T?
+U 1 1 5EA02F3C
+P 4000 5450
+F 0 "T?" H 3683 5815 50  0000 C CNN
+F 1 "ACJS-MHDR" H 3683 5724 50  0000 C CNN
+F 2 "AVR-KiCAD-Lib-Connectors:ACJS-MHDR" H 3900 6950 50  0001 C CNN
+F 3 "https://www.amphenol-sine.com/pdf/datasheet/ACJS-MHDR.pdf" H 4000 7050 50  0001 C CNN
+F 4 "1.41000" H 4200 7200 50  0001 C CNN "Cost QTY: 1"
+F 5 "0.81420" H 4300 7300 50  0001 C CNN "Cost QTY: 1000"
+F 6 "0.74520" H 4400 7400 50  0001 C CNN "Cost QTY: 2500"
+F 7 "*" H 4500 7500 50  0001 C CNN "Cost QTY: 5000"
+F 8 "*" H 4600 7600 50  0001 C CNN "Cost QTY: 10000"
+F 9 "Amphenol Sine Systems Corp" H 4700 7700 50  0001 C CNN "MFR"
+F 10 "ACJS-MHDR" H 4800 7800 50  0001 C CNN "MFR#"
+F 11 "Digikey" H 4900 7900 50  0001 C CNN "Vendor"
+F 12 "889-1817-ND" H 5000 8000 50  0001 C CNN "Vendor #"
+F 13 "AVR" H 5100 8100 50  0001 C CNN "Designer"
+F 14 "12.7mm" H 5200 8200 50  0001 C CNN "Height"
+F 15 "1/5/2019" H 6300 9300 50  0001 C CNN "Date Created"
+F 16 "1/5/2019" H 5300 8300 50  0001 C CNN "Date Modified"
+F 17 "Yes" H 5400 8400 50  0001 C CNN "Lead-Free ?"
+F 18 "RoHS 1" H 5500 8500 50  0001 C CNN "RoHS Levels"
+F 19 "ThroughHole" H 5600 8600 50  0001 C CNN "Mounting"
+F 20 "6" H 5700 8700 50  0001 C CNN "Pin Count #"
+F 21 "Active" H 5800 8800 50  0001 C CNN "Status"
+F 22 "*" H 5900 8900 50  0001 C CNN "Tolerance"
+F 23 "TRS Connector 6.35mm" H 6000 9000 50  0001 C CNN "Type"
+F 24 "*" H 6100 9100 50  0001 C CNN "Voltage"
+F 25 "*" H 6200 9250 50  0001 C CNN "Package"
+F 26 "CONN JACK STEREO 1/4\" R/A" H 6600 9650 50  0001 C CNN "Description"
+F 27 "ACJS-MHDR" H 6400 9450 50  0001 C CNN "_Value_"
+F 28 "*" H 6500 9550 50  0001 C CNN "Management_ID"
+	1    4000 5450
+	1    0    0    -1
+$EndComp
 $EndSCHEMATC
