File: PCB/X0chimilc0/USB_C.sch (KiCad schematic (older format))
At the start: 46 parts

Commit message: USB C DDR3L MCU
more with MCU and USB C and DDR3L
Connections:
- net USB_C1_D+: now reaches T?.A6 (D+), T?.B6 (D+)
- net USB_C1_D-: now reaches T?.A7 (D-), T?.B7 (D-)
- net USB_C2_D+: now reaches T?.A6 (D+), T?.B6 (D+)
- net USB_C2_D-: now reaches T?.A7 (D-), T?.B7 (D-)
Other:
- note added: "PA11"
- note added: "PA12"
- note added: "PA9"
- note added: "PB13"
- note added: "PB14"
- note added: "PB15"
- note added: "USB Device & Host/OTG Over USB - C"
- moved on the sheet: C?, Q?A, Q?B, R?, T?, U?
