File: PCB/X0chimilc0/FPGA.sch (KiCad schematic (older format))
At the start: 2 parts, among them U2 ECP5UM5G_85_CABGA381

Commit message: Memory
Memory Symbol and footprint designed and added to schematic
Parts:
- gave numbers to parts that had none: 1
Changed lines of the file:
@@
 EESchema Schematic File Version 4
+LIBS:X0chimilc0-cache
 EELAYER 30 0
 EELAYER END
@@
 $EndComp
 $Comp
-L Connector_Generic:Conn_02x12_Odd_Even J?
+L Connector_Generic:Conn_02x12_Odd_Even J1
 U 1 1 5E4F1C5B
 P 3150 10050
-F 0 "J?" H 3200 10767 50  0000 C CNN
+F 0 "J1" H 3200 10767 50  0000 C CNN
 F 1 "Conn_02x12_Odd_Even" H 3200 10676 50  0000 C CNN
 F 2 "Connectors_Harwin:Harwin_LTek-Male_2x13x2.00mm_Straight_StrainRelief" H 3150 10050 50  0001 C CNN

Commit message: Component PDFs
added relevant PDF datasheets and some minor schematic edits
Parts:
- removed J1: Conn_02x12_Odd_Even, Connectors_Harwin:Harwin_LTek-Male_2x13x2.00mm_Straight_StrainRelief, symbol Connector_Generic:Conn_02x12_Odd_Even
Changed lines of the file:
@@
-	1    0    0    -1
-$EndComp
-$Comp
-L Connector_Generic:Conn_02x12_Odd_Even J1
-U 1 1 5E4F1C5B
-P 3150 10050
-F 0 "J1" H 3200 10767 50  0000 C CNN
-F 1 "Conn_02x12_Odd_Even" H 3200 10676 50  0000 C CNN
-F 2 "Connectors_Harwin:Harwin_LTek-Male_2x13x2.00mm_Straight_StrainRelief" H 3150 10050 50  0001 C CNN
-F 3 "~" H 3150 10050 50  0001 C CNN
-	1    3150 10050
 	1    0    0    -1
 $EndComp

Commit message: USB C DDR3L MCU
more with MCU and USB C and DDR3L
Parts:
- removed U2: ECP5UM5G_85_CABGA381, AVR-KiCAD-Lib-ICs:381caBGA_LATTICE, symbol AVR-KiCAD-Lib-ICs:ECP5UM5G_85_CABGA381
